File: Hardware/Hardware.kicad_sch (KiCad schematic)
At the start: 0 parts

Commit message: 添加MCU
Parts:
- added U1: GD32F470VIT6, kicad_api_lib:GD32F470VIT6, symbol GD32F470VIT6:GD32F470VIT6
- added U2: USB3300-EZK, kicad_api_lib:USB3300-EZK, symbol USB3300-EZK:USB3300-EZK
Connections:
- new net +1V8: U2.15 (VDD1.8), U2.26 (VDD1.8), U2.29 (VDDA1.8)
- new net +3.3V: U2.16 (VDD3.3), U2.25 (VDD3.3), U2.30 (VDD3.3), U2.6 (VDD3.3)
- new net +3.3VA: U1.22 (VDDA)
- new net GND: U2.1 (GND), U2.2 (GND), U2.33 (GND)
- new net GNDA: U1.20 (VSSA)
- new net USB_CK: U2.14 (CLKOUT)
- new net USB_D0: U2.24 (DATA0)
- new net USB_D1: U2.23 (DATA1)
- new net USB_D2: U2.22 (DATA2)
- new net USB_D3: U2.21 (DATA3)
- new net USB_D4: U2.20 (DATA4)
- new net USB_D5: U2.19 (DATA5)
- new net USB_D6: U2.18 (DATA6)
- new net USB_D7: U2.17 (DATA7)
- new net USB_DIR: U2.12 (DIR)
- new net USB_NXT: U2.11 (NXT)
- new net USB_RESET: U2.9 (RESET)
- new net USB_STP: U2.13 (STP)
